File: aristotle_split_33_keyboard-2021.kicad_pcb (KiCad board)
At the start: 2 copper layers, 257.6 x 96.8 mm, 85 parts, among them J1 8P8C, J2 8P8C, J3 Conn_01x02_Male, K11 SW_PUSH, K12 SW_PUSH, K13 SW_PUSH, K14 SW_PUSH, K15 SW_PUSH, K16 SW_PUSH, K17 SW_PUSH, K18 SW_PUSH, K19 SW_PUSH, K1A1 SW_PUSH, K21 SW_PUSH, K22 SW_PUSH, K23 SW_PUSH, K24 SW_PUSH, K25 SW_PUSH, K26 SW_PUSH, K27 SW_PUSH, K28 SW_PUSH, K29 SW_PUSH, K2A1 SW_PUSH, K31 SW_PUSH, K32 SW_PUSH, K33 SW_PUSH, K34 SW_PUSH, K35 SW_PUSH, K36 SW_PUSH, K37 SW_PUSH, K38 SW_PUSH, K39 SW_PUSH, K3A1 SW_PUSH, K45 SW_PUSH, K49 SW_PUSH, K4A1 SW_PUSH, SW1 SW_SPDT, U1 ProMicro

Commit message: Create case
Parts:
- removed 3: MountingHole_2.2mm_M2, MountingHole:MountingHole_2.2mm_M2
- removed the breakaway at (178.2, 108.2)
- removed the breakaway at (175.0, 108.2)
- J3: footprint Connector_JST:JST_XH_B2B-XH-A_1x02_P2.50mm_Vertical -> Connector_PinHeader_2.54mm:PinHeader_1x02_P2.54mm_Vertical_SMD_Pin1Left
- U1: value ProMicro -> ProMicro_r
- moved D1A1 10.9 mm to (79.8, 99.6), turned to 90 degrees
- moved D14 10.2 mm to (235.6, 96.9), turned to 90 degrees
- moved D18 10.2 mm to (117.5, 89.9), turned to 90 degrees
- moved D15 10.2 mm to (254.6, 98.9), turned to 90 degrees
- moved D29 10.2 mm to (98.5, 114.9), turned to 90 degrees
- moved D28 10.2 mm to (117.5, 107.9), turned to 90 degrees
- moved D27 8.97 mm to (136.5, 111.7), turned to 90 degrees
- moved D19 7.49 mm to (98.5, 94.2), turned to 90 degrees
- moved D17 5.58 mm to (136.5, 94.9), turned to 90 degrees
- moved D38 3.37 mm to (117.5, 119.2)
- moved D23 3.35 mm to (216.6, 101.2)
- moved D21 2.91 mm to (197.6, 114.7)
- moved J3 2.02 mm to (71.1, 115.7)
- moved D33 1.82 mm to (216.6, 124.4)
- moved D22 1.50 mm to (197.6, 101.2)
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- renumbered RESET to RESET1
Connections:
- D11 pad 1: row11 -> row13
- D15 pad 1: row11 -> row10
- D21 pad 1: row12 -> row13
- D24 pad 1: row12 -> row11
- D25 pad 1: row12 -> row11
- D33 pad 1: row13 -> row12
- D34 pad 1: row13 -> row12
- D35 pad 1: row13 -> row12
- D45 pad 1: row10 -> row13
- J1 pad : GND -> (no net)
- J1 pad 1: row0 -> col0
- J1 pad 2: col3 -> row0
- J1 pad 3: row1 -> col1
- J1 pad 4: col0 -> row3
- J1 pad 5: row2 -> col2
- J1 pad 6: col2 -> row2
- J1 pad 7: col1 -> col3
- J1 pad 8: row3 -> row1
- J2 pad 1: row10 -> col10
- J2 pad 2: col13 -> row10
- J2 pad 3: row11 -> col11
- J2 pad 4: col10 -> row13
- J2 pad 5: row12 -> col12
- J2 pad 6: col12 -> row12
- J2 pad 7: col11 -> col13
- J2 pad 8: row13 -> row11
- K11 pad 1: col10 -> col11
- K22 pad 1: col11 -> col10
- K23 pad 1: col12 -> col11
- K31 pad 1: col10 -> col12
- K32 pad 1: col11 -> col10
- U1 pad 10: col2 -> row2
- U1 pad 11: col1 -> col3
- U1 pad 12: row3 -> row1
- U1 pad 13: (no net) -> col6
- U1 pad 14: (no net) -> col5
- U1 pad 15: col8 -> col4
- U1 pad 16: col7 -> row0
- U1 pad 17: col6 -> (no net)
- U1 pad 18: col5 -> (no net)
- U1 pad 19: col4 -> (no net)
- U1 pad 2: (no net) -> col7
- U1 pad 20: row0 -> (no net)
- U1 pad 5: (no net) -> col8
- U1 pad 6: col3 -> col0
- U1 pad 7: row1 -> col1
- U1 pad 8: col0 -> row3
- U1 pad 9: row2 -> col2
Routing:
- net col12: track 98.8 -> 168.9 mm
- net row10: track 133.8 -> 89.7 mm
- net col7: track 114.8 -> 158.7 mm
- net row11: track 129.5 -> 89.5 mm
- net col8: track 142.3 -> 174.2 mm
- net col11: track 136.7 -> 167.9 mm
- net row13: track 102.7 -> 130.6 mm
- net row12: track 114.2 -> 91.3 mm
- net col10: track 155.1 -> 172.9 mm
- net col13: track 100.1 -> 117.6 mm
- net row0: track 128.3 -> 111.0 mm
- net row1: track 144.8 -> 131.8 mm
- net col5: track 105.4 -> 117.6 mm
- net row3: track 53.8 -> 65.8 mm
- net col3: track 36.7 -> 27.2 mm
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Other:
- outline, holes or cut-outs redrawn
- net class Power added: clearance 0.2, trace_width 0.5, via_dia 1, via_drill 0.5
- rule pad_to_mask_clearance: 0.051 -> 0
