File: aristotle_split_33_keyboard-2021.sch (KiCad schematic (older format))
At the start: 78 parts, among them J1 8P8C, J2 8P8C, J3 Conn_01x02_Male, K11 SW_PUSH, K12 SW_PUSH, K13 SW_PUSH, K14 SW_PUSH, K15 SW_PUSH, K16 SW_PUSH, K17 SW_PUSH, K18 SW_PUSH, K19 SW_PUSH, K1A1 SW_PUSH, K21 SW_PUSH, K22 SW_PUSH, K23 SW_PUSH, K24 SW_PUSH, K25 SW_PUSH, K26 SW_PUSH, K27 SW_PUSH, K28 SW_PUSH, K29 SW_PUSH, K2A1 SW_PUSH, K31 SW_PUSH, K32 SW_PUSH, K33 SW_PUSH, K34 SW_PUSH, K35 SW_PUSH, K36 SW_PUSH, K37 SW_PUSH, K38 SW_PUSH, K39 SW_PUSH, K3A1 SW_PUSH, K45 SW_PUSH, K49 SW_PUSH, K4A1 SW_PUSH, SW1 SW_SPDT, U1 ProMicro_r

Commit message: Create case
Parts:
- J3: footprint Connector_JST:JST_XH_B2B-XH-A_1x02_P2.50mm_Vertical -> Connector_PinHeader_2.54mm:PinHeader_1x02_P2.54mm_Vertical_SMD_Pin1Left
- K11, K12, K13, K14, K15, K16, K17, K18, K19, K1A1, K21, K22, K23, K24, K25, K26, K27, K28, K29, K2A1, K31, K32, K33, K34, K35, K36, K37, K38, K39, K3A1, K45, K49, K4A1: footprint aristotle:Kailh-Choc_v2-Keyswitch -> aristotle:Kailh-Choc_1350-Keyswitch-NONREVERSIBLE
Connections:
- net col0: now also J1.1, U1.6 (D0/SCL); no longer J1.4, U1.8 (C6)
- net col1: now also J1.3, U1.7 (D4); no longer J1.7, U1.11 (B4)
- net col10: now also J2.1, K22.1, K32.1; no longer J2.4, K11.1, K31.1
- net col11: now also J2.3, K11.1, K23.1; no longer J2.7, K22.1, K32.1
- net col12: now also J2.5, K31.1; no longer J2.6, K23.1
- net col13: now also J2.7; no longer J2.2
- net col2: now also J1.5, U1.9 (D7); no longer J1.6, U1.10 (E6)
- net col3: now also J1.7, U1.11 (B4); no longer J1.2, U1.6 (D0/SCL)
- net col4: now also U1.15 (B3); no longer U1.19 (F5)
- net col5: now also U1.14 (B2); no longer U1.18 (F6)
- net col6: now also U1.13 (B6); no longer U1.17 (F7)
- net col7: now also U1.2 (D2/RX); no longer U1.16 (B1)
- net col8: now also U1.5 (D1/SDA); no longer U1.15 (B3)
- net row0: now also J1.2, U1.16 (B1); no longer J1.1, U1.20 (F4)
- net row1: now also J1.8, U1.12 (B5); no longer J1.3, U1.7 (D4)
- net row10: now also D15.1 (K), J2.2; no longer D45.1 (K), J2.1
- net row11: now also D24.1 (K), D25.1 (K), J2.8; no longer D11.1 (K), D15.1 (K), J2.3
- net row12: now also D33.1 (K), D34.1 (K), D35.1 (K), J2.6; no longer D21.1 (K), D24.1 (K), D25.1 (K), J2.5
- net row13: now also D11.1 (K), D21.1 (K), D45.1 (K), J2.4; no longer D33.1 (K), D34.1 (K), D35.1 (K), J2.8
- net row2: now also J1.6, U1.10 (E6); no longer J1.5, U1.9 (D7)
- net row3: now also J1.4, U1.8 (C6); no longer J1.8, U1.12 (B5)
Other:
- moved on the sheet: D11, D15, D21, D22, D23, D24, D25, D31, D32, D33, D34, D35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
